File: kicad_rev-/esp32hardware.kicad_pcb (KiCad board)
At the start: 2 copper layers, 40 parts, among them U1 TS4231, U2 TS4231, U3 TS4231, U4 TS4231, U5 TS4231, U6 TS4231, U7 TS4231, U8 TS4231

Commit message: More progress...
Parts:
- added C17: .1uF, C_0603, F.Cu at (134.0, 71.0)
- added C18: .1uF, C_0603, F.Cu at (162.0, 75.0)
- added C19: .1uF, C_0603, F.Cu at (47.0, 90.9)
- added C20: .1uF, C_0603, F.Cu at (74.1, 77.5)
- added C21: .1uF, C_0603, F.Cu at (70.1, 74.4)
- added C22: 1uF, C_0603, F.Cu at (143.0, 85.0)
- added C23: .1uF, C_0603, F.Cu at (162.5, 69.5)
- added C24: 10uF, C_0603, F.Cu at (31.5, 112.6)
- added C25: 10uF, C_0603, F.Cu at (56.7, 79.0)
- added C26: 10uF, C_0603, F.Cu at (62.1, 74.2)
- added C27: 22uF, C_0603, F.Cu at (47.1, 67.4)
- added C28: 22uF, C_0603, F.Cu at (52.1, 82.5)
- added D9: D_Schottky, D_SOD-123, F.Cu at (165.5, 85.0)
- added J1: AUX_HEADER, RIBBON12SMT, F.Cu at (155.0, 94.0)
- added J2: BAT1, Pin_Header_Straight_1x02_Pitch2.54mm, F.Cu at (133.5, 85.0)
- added J3: BAT2, Pin_Header_Straight_1x02_Pitch2.54mm, F.Cu at (173.0, 75.0)
- added P1: USB, USBMicroB-10118194-0001LF, F.Cu at (178.0, 90.0)
- added P3: WSOUT, Pin_Header_Straight_1x03_Pitch2.54mm, F.Cu at (106.0, 135.5)
- added Q1: SS8050, SOT-23, F.Cu at (173.0, 100.0)
- added Q2: SS8050, SOT-23, F.Cu at (169.0, 100.0)
- added Q3: SSM3J355RLFCT-ND, SOT-23, F.Cu at (162.5, 113.0)
- added Q4: SS8050, SOT-23, F.Cu at (38.8, 122.4)
- added Q5: SSM3J355RLFCT-ND, SOT-23, F.Cu at (31.5, 90.5)
- added R10: 10k, R_0603, F.Cu at (167.0, 97.0)
- added R11: 10k, R_0603, F.Cu at (170.0, 86.0)
- added R12: 10k, R_0603, F.Cu at (45.7, 85.2)
- added R13: 10k, R_0603, F.Cu at (58.0, 83.7)
- added R14: 3.3k, R_0603, F.Cu at (138.0, 44.0)
- added R15: 3.3k, R_0603, F.Cu at (59.9, 78.5)
- added R16: 3.3k, R_0603, F.Cu at (77.3, 73.1)
- added R17: 3.3k, R_0603, F.Cu at (60.1, 71.5)
- added R18: 15k, R_0603, F.Cu at (42.7, 88.6)
- added R19: 1M, R_0603, F.Cu at (40.8, 83.7)
- added R20: 1M, R_0603, F.Cu at (139.0, 75.0)
- added R21: 1M, R_0603, F.Cu at (48.4, 86.9)
- added R22: 1M, R_0603, F.Cu at (138.0, 72.0)
- added R23: 1M, R_0603, F.Cu at (51.5, 76.9)
- added R24: 10k, R_0603, F.Cu at (42.5, 78.8)
- added R25: 10k, R_0603, F.Cu at (65.7, 79.8)
- added R26: 10k, R_0603, F.Cu at (65.5, 82.6)
- added R27: 10k, R_0603, F.Cu at (150.0, 47.0)
- added R28: 10k, R_0603, F.Cu at (149.0, 44.0)
- added R29: 10k, R_0603, F.Cu at (69.9, 79.8)
- added R9: 10k, R_0603, F.Cu at (51.0, 101.0)
- added REF**: Pin_Header_Straight_1x03_Pitch2.54mm, Pin_Headers:Pin_Header_Straight_1x03_Pitch2.54mm, F.Cu at (196.0, 76.0)
- added REF**: Pin_Header_Straight_1x02_Pitch2.54mm, Pin_Headers:Pin_Header_Straight_1x02_Pitch2.54mm, F.Cu at (193.0, 64.0)
- added SW1: TACTILE, TACTILE10, F.Cu at (172.0, 113.0)
- added U10: MCP1824v3.3, SOT-23-5, F.Cu at (134.0, 76.0)
- added U11: MCP1824v2.5, SOT-23-5, F.Cu at (161.5, 67.0)
- added U12: STBC08, DFN6PAD, F.Cu at (144.0, 88.5)
- added U13: LSM303C, 12LGA, F.Cu at (160.0, 72.0)
- added U14: ESP32-WROOM, ESP32-WROOM, F.Cu at (132.0, 59.0)
- added U9: CP2102, QFN-24-1EP_4x4mm_Pitch0.5mm, F.Cu at (169.0, 91.0)
- moved C1 111.7 mm to (29.5, 24.9)
- moved C10 111.7 mm to (42.0, 24.9)
- moved C11 111.7 mm to (52.0, 24.9)
- moved C12 111.7 mm to (62.0, 24.9)
- moved C15 111.7 mm to (91.5, 24.9)
- moved C16 111.7 mm to (101.5, 24.9)
- moved C2 111.7 mm to (38.0, 24.9)
- moved C3 111.7 mm to (48.0, 24.9)
- moved C4 111.7 mm to (58.0, 24.9)
- moved C7 111.7 mm to (87.5, 24.9)
- moved C8 111.7 mm to (96.0, 24.9)
- moved C9 111.7 mm to (33.5, 24.9)
- moved D1 111.7 mm to (33.0, 21.4)
- moved D2 111.7 mm to (42.5, 21.4)
- moved D3 111.7 mm to (52.0, 21.4)
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Connections:
- U1 pad C1: (no net) -> D0
- U1 pad C2: (no net) -> E0
- U2 pad C1: (no net) -> D1
- U2 pad C2: (no net) -> E1
- U3 pad C1: (no net) -> D2
- U3 pad C2: (no net) -> E2
- U4 pad C1: (no net) -> D3
- U4 pad C2: (no net) -> E3
- U5 pad C1: (no net) -> D4
- U5 pad C2: (no net) -> E4
- U6 pad C1: (no net) -> D5
- U6 pad C2: (no net) -> E5
- U7 pad C1: (no net) -> D6
- U7 pad C2: (no net) -> E6
- U8 pad C1: (no net) -> D7
- U8 pad C2: (no net) -> E7
Routing:
- net +5V: track 0.00 -> 15.2 mm, vias 0 -> 2
- net GND: track 28.0 -> 38.1 mm
- net +3V3: track 13.2 -> 22.5 mm
- net Net-(P1-Pad3): track 0.00 -> 5.95 mm, vias 0 -> 2
- net +2.5V: track 0.00 -> 4.77 mm
- net Net-(P1-Pad2): track 0.00 -> 4.39 mm
- net Net-(R11-Pad1): track 0.00 -> 3.05 mm
- net Net-(C18-Pad1): track 0.00 -> 2.81 mm
- net (no net): track 36.1 -> 35.3 mm
Other:
- board outline added: 50 x 110 mm
- board text added: "+Y"
